Commit message: IMU pose publishing

File: catkin_ws/src/grapebot_gazebo_sim/urdf/grapebot_lite_assy_controllers.urdf (robot description, URDF)
Before this commit: robot grapebot, 8 links, 7 joints
Joints:
- joint back_right_wheel_joint: limit effort=100.0 velocity=100.0 -> effort=1000.0 velocity=1000.0
- joint front_wheel_axis_joint: limit lower=-0.78 upper=0.78 effort=100.0 velocity=100.0 -> lower=-0.78 upper=0.78 effort=1000.0 velocity=1000.0
- joint front_wheel_joint: limit effort=100.0 velocity=100.0 -> effort=1000.0 velocity=1000.0
